File: mcu.kicad_sch (KiCad schematic)
At the start: 50 parts, among them J1 I2C EKRAN, SW1 SW_Push, SW2 SW_Push, U1 STM32F205VGTx, U12 TMP101, Y1 8MHz

Commit message: LAST I HOPE
Connections:
- net PANIC STOP: now reaches U1.46 (PE15)
- net Current Sense_C: now reaches U1.67 (PA8)
- net Current_Sense_A renamed Current Sense_A
- net Current_Sense_B renamed Current Sense_B
- no-connect marks 44 -> 42
Changed lines of the file:
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@@
-	)
-	(no_connect
-		(at 124.46 72.39)
 	)
 	(no_connect
@@
 	(no_connect
 		(at 124.46 146.05)
-	)
-	(no_connect
-		(at 73.66 113.03)
 	)
 	(no_connect
@@
 		)
 	)
-	(global_label "Current_Sense_B"
+	(global_label "Current Sense_B"
 		(shape input)
 		(at 124.46 69.85 0)
@@
 		)
 	)
+	(global_label "PANIC STOP"
+		(shape input)
+		(at 73.66 113.03 180)
+		(fields_autoplaced yes)
+		(effects
+			(font
+				(size 1.27 1.27)
+			)
+			(justify right)
+		)
+		(property "Intersheetrefs" "${INTERSHEET_REFS}"
+			(at 59.3657 113.03 0)
+			(effects
+				(font
+					(size 1.27 1.27)
+				)
+				(justify right)
+				(hide yes)
+			)
+		)
+	)
 	(global_label "BT_RX"
 		(shape input)
@@
 		)
 	)
-	(global_label "Current_Sense_A"
+	(global_label "Current Sense_A"
 		(shape input)
 		(at 124.46 67.31 0)
@@
 			(effects
 				(font
+					(size 1.27 1.27)
+				)
+				(justify left)
+				(hide yes)
+			)
+		)
+	)
+	(global_label "Current Sense_C"
+		(shape input)
+		(at 124.46 72.39 0)
+		(fields_autoplaced yes)
+		(effects
+			(font
+				(size 1.27 1.27)
+			)
+			(justify left)
+		)
+		(property "Intersheetrefs" "${INTERSHEET_REFS}"
+			(at 143.1689 72.39 0)
+			(effects
+				(font

Commit message: son update
Changed lines of the file:
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@@
 		(on_board yes)
 		(dnp no)
-		(fields_autoplaced yes)
 		(property "Reference" "#FLG05"
 			(at 111.76 34.925 0)
@@
 		)
 		(property "Value" "PWR_FLAG"
-			(at 111.76 31.75 0)
+			(at 114.808 31.242 0)
 			(effects
 				(font
