File: mcu.kicad_sch (KiCad schematic)
At the start: 44 parts, among them J1 I2C EKRAN, SW1 SW_Push, SW2 SW_Push, U1 STM32G474VETx, U12 TMP101, Y1 8MHz

Commit message: rev3
Parts:
- removed R23: 100, Resistor_SMD:R_0603_1608Metric_Pad0.98x0.95mm_HandSolder, symbol Device:R
- removed R24, R25: 4.7K, Resistor_SMD:R_0603_1608Metric_Pad0.98x0.95mm_HandSolder, symbol Device:R
- removed U12: TMP101, Package_TO_SOT_SMD:SOT-23-6, symbol Sensor_Temperature:TMP101
- C28: footprint Capacitor_THT:C_Disc_D10.5mm_W5.0mm_P5.00mm -> Resistor_SMD:R_0805_2012Metric_Pad1.20x1.40mm_HandSolder
- R7: footprint Resistor_THT:R_Axial_DIN0207_L6.3mm_D2.5mm_P7.62mm_Horizontal -> Resistor_SMD:R_1210_3225Metric
Connections:
- net ACCEL: now also U1.46 (PE15); no longer U1.22 (PA2)
- net BOOT0: now also U1.96 (PB9); no longer U1.95 (PB8)
- net BRAKE: now also U1.45 (PE14); no longer U1.1 (PE2)
- net BUZZER: now also U1.87 (PD5); no longer U1.97 (PE0)
- net Current Sense_A: now also U1.32 (PB0); no longer U1.28 (PA6)
- net Current_Sense_C: now also U1.52 (PB13); no longer U1.32 (PB0)
- net HALL_A: now also U1.59 (PD12); no longer U1.65 (PC6)
- net HALL_B: now also U1.57 (PD10); no longer U1.66 (PC7)
- net HALL_C: now also U1.55 (PD8); no longer U1.67 (PC8)
- net HS_MOS_A: now also U1.39 (PE8); no longer U1.40 (PE9)
- net HS_MOS_B: now also U1.41 (PE10); no longer U1.42 (PE11)
- net HS_MOS_C: now also U1.43 (PE12); no longer U1.44 (PE13)
- net I2C_SCL: now also U1.95 (PB8); no longer U1.93 (PB6)
- net I2C_SDA: now also U1.78 (PA15); no longer U1.94 (PB7)
- net LS_MOS_A: now also U1.40 (PE9); no longer U1.39 (PE8)
- net LS_MOS_B: now also U1.42 (PE11); no longer U1.41 (PE10)
- net LS_MOS_C: now also U1.44 (PE13); no longer U1.43 (PE12)
- net PANIC STOP: now also U1.7 (PC13); no longer U1.46 (PE15)
- net REGEN: now also U1.70 (PA9); no longer U1.26 (PA4)
- net STATUS_LED: now also U1.90 (PB3); no longer U1.98 (PE1)
- net TEMP_SENSOR: now also U1.69 (PA8); no longer U1.25 (PA3)
- net BT_KEY: no longer names the net of U1.51 (PB12)
- net BT_RX: no longer names the net of U1.50 (PB11)
- net BT_STATE: no longer names the net of U1.68 (PC9)
- net BT_TX: no longer names the net of U1.47 (PB10)
- net B_VOL_CHECK: no longer names the net of U1.21 (PA1)
- net CSense_OUT_LES: no longer names the net of U1.20 (PA0)
- net TMP_ALERT: no longer names the net of U1.18 (PC3)
- net TMP_SCL: no longer names the net of U1.16 (PC1)
- net TMP_SDA: no longer names the net of U1.15 (PC0)
- no-connect marks 47 -> 59
Other:
- note added: "TIM1 HATLARI"
- moved on the sheet: J1, R10, R9
