File: Motor_Driver_Shell_Eco.kicad_pcb (KiCad board)
At the start: 2 copper layers, 149 parts, among them J1 I2C EKRAN, J10 Conn_01x02, J2 HALL INPUT, J3 Conn_01x02, J4 Conn_01x01, J5 Conn_01x04, J6 Conn_01x06, J7 Conn_01x02, J8 Conn_01x03, J9 Conn_01x03, P1 TYPE_C Receptacle, Q1 BC817, Q10 IXTP90N15T, Q11 IXTP90N15T, Q12 IXTP90N15T, Q13 IXTP90N15T, Q2 IXTP90N15T, Q3 IXTP90N15T, Q4 IXTP90N15T, Q5 IXTP90N15T, Q6 IXTP90N15T, Q7 IXTP90N15T, Q8 IXTP90N15T, Q9 IXTP90N15T, SW1 SW_Push, SW2 SW_Push, U1 STM32F205VGTx, U2 LM5017MR, U3 AP2204K-5.0, U4 XC6206 - 3V3, U5 IR2110, U6 IR2110, U7 IR2110, U8 TJA1051T, Y1 8MHz

Commit message: LATEST UPDATES
Parts:
- C18, C19, C20, C21, C22, C23, C24: footprint Capacitor_SMD:C_1210_3225Metric_Pad1.33x2.70mm_HandSolder -> Capacitor_SMD:C_0603_1608Metric_Pad1.08x0.95mm_HandSolder
- C25: footprint Capacitor_THT:C_Radial_D12.5mm_H25.0mm_P5.00mm -> Capacitor_SMD:C_0603_1608Metric_Pad1.08x0.95mm_HandSolder
- C26: footprint Capacitor_THT:C_Disc_D10.5mm_W5.0mm_P5.00mm -> Capacitor_SMD:C_0603_1608Metric_Pad1.08x0.95mm_HandSolder
- C27: value C -> 10uf; footprint Capacitor_THT:C_Radial_D6.3mm_H5.0mm_P2.50mm -> Capacitor_SMD:C_0805_2012Metric_Pad1.18x1.45mm_HandSolder
- C31, C32: footprint Capacitor_THT:C_Rect_L7.2mm_W8.5mm_P5.00mm_FKP2_FKP2_MKS2_MKP2 -> Capacitor_SMD:C_0603_1608Metric_Pad1.08x0.95mm_HandSolder
- J4: value Conn_01x01 -> Conn_01x02; footprint Connector_PinSocket_1.27mm:PinSocket_1x01_P1.27mm_Vertical -> Connector_PinSocket_2.00mm:PinSocket_1x02_P2.00mm_Vertical
- S1: footprint Resistor_THT:R_Axial_DIN0207_L6.3mm_D2.5mm_P7.62mm_Horizontal -> LES-50NP:LES50NP
- moved C3 330.1 mm to (398.6, 116.4), turned to 180 degrees
- moved C2 319.9 mm to (390.6, 138.9), turned to 90 degrees
- moved C1 304.1 mm to (374.1, 140.2), turned to 90 degrees
- moved C4 298.7 mm to (384.6, 122.9), turned to 180 degrees
- moved C6 289.6 mm to (375.1, 122.4), turned to 180 degrees
- moved C5 289.5 mm to (375.1, 115.4), turned to 180 degrees
- moved R1 276.8 mm to (361.6, 141.1), turned to 90 degrees
- moved D1 264.3 mm to (358.1, 140.5), turned to 90 degrees
- moved S1 262.2 mm to (353.7, 128.7), turned to -90 degrees
- moved R2 257.0 mm to (349.6, 126.1), turned to 90 degrees
- moved F1 255.6 mm to (335.4, 168.7), turned to 90 degrees
- moved R12 254.4 mm to (368.2, 65.8)
- moved H2 252.1 mm to (337.1, 121.9), turned to 90 degrees
- moved R11 251.7 mm to (366.1, 64.1), turned to 180 degrees
- moved H1 249.2 mm to (335.4, 176.5), turned to 90 degrees
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Connections:
- C11 pad 2: -VDC -> GND
- C12 pad 2: -VDC -> GND
- C13 pad 2: -VDC -> GND
- C14 pad 2: -VDC -> GND
- C18 pad 1: -VDC -> GND
- C19 pad 1: -VDC -> GND
- C20 pad 1: -VDC -> GND
- C21 pad 1: -VDC -> GND
- C22 pad 1: -VDC -> GND
- C23 pad 1: -VDC -> GND
- C24 pad 1: -VDC -> GND
- C25 pad 2: -VDC -> GND
- C26 pad 2: -VDC -> GND
- C27 pad 2: -VDC -> GND
- C28 pad 1: -VDC -> GND
- C29 pad 1: -VDC -> GND
- C30 pad 1: -VDC -> GND
- C31 pad 2: -VDC -> GND
- C32 pad 2: -VDC -> GND
- C33 pad 2: -VDC -> GND
- C34 pad 2: -VDC -> GND
- C35 pad 2: -VDC -> GND
- C45 pad 2: -VDC -> GND
- C7 pad 2: -VDC -> GND
- C8 pad 2: -VDC -> GND
- C9 pad 2: -VDC -> GND
- D3 pad 1: -VDC -> GND
- J1 pad 4: -VDC -> GND
- J10 pad 1: -VDC -> GND
- J2 pad 5: -VDC -> GND
- J4 pad 1: -VDC -> GND
- J5 pad 3: -VDC -> GND
- J6 pad 4: -VDC -> GND
- J7 pad 1: -VDC -> GND
- J8 pad 3: -VDC -> GND
- J9 pad 3: -VDC -> GND
- P1 pad A1: -VDC -> GND
- P1 pad A12: -VDC -> GND
- P1 pad B1: -VDC -> GND
- P1 pad B12: -VDC -> GND
- P1 pad S1: -VDC -> GND
- Q1 pad 2: -VDC -> GND
- R5 pad 1: -VDC -> GND
- R50 pad 2: -VDC -> TEMP_SENSOR
- R51 pad 1: -VDC -> GND
- R52 pad 1: -VDC -> GND
- R8 pad 2: -VDC -> GND
- SW1 pad 1: -VDC -> GND
- U1 pad 10: -VDC -> GND
- U1 pad 20: -VDC -> GND
- U1 pad 27: -VDC -> GND
- U1 pad 74: -VDC -> GND
- U3 pad 2: -VDC -> GND
- U4 pad 1: -VDC -> GND
- U5 pad 13: -VDC -> GND
- U6 pad 13: -VDC -> GND
- U7 pad 13: -VDC -> GND
- U8 pad 2: -VDC -> GND
- U8 pad 8: -VDC -> GND
Routing:
- net -VDC: track 0.00 -> 119.9 mm
- net +VDC: track 0.00 -> 117.0 mm
- net /MCU/NRST: track 0.00 -> 36.0 mm
- net Net-(F1-Pad2): track 0.00 -> 30.0 mm
- net /MCU/I2C_SCL: track 0.00 -> 21.9 mm
- net +3V3: track 0.00 -> 21.4 mm
- net /MCU/I2C_SDA: track 0.00 -> 20.0 mm
- net STATUS_LED: track 0.00 -> 16.2 mm
- net Net-(U1-PH0): track 0.00 -> 15.1 mm
- net Net-(U1-PH1): track 0.00 -> 15.1 mm
- net GND: track 0.00 -> 13.1 mm
- net Net-(F1-Pad1): track 0.00 -> 13.0 mm
- net /MCU/BOOT0: track 0.00 -> 10.2 mm
- net BUZZER: track 0.00 -> 8.65 mm
- net VREF+: track 0.00 -> 8.43 mm
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- added copper zone on F.Cu, net GND
- added copper zone on In1.Cu, net GND
Other:
- copper layers 2 -> 6

Commit message: Fet Drivers  olarak IRS21867S, MOSFET olarak IAUS300N08S5N014 değiştirildi. Decoupler kısmı değiştirildi, (paraziter direnci arttırıldı.) buzzer düzeltildi ve utility kısmına alındı. CAN-BUS bitti. LDO sayısı 2x oldu
Parts:
- moved C8 204.9 mm to (318.4, 176.6), turned to -90 degrees
- moved C7 167.3 mm to (327.4, 176.7), turned to -90 degrees
- moved C3 67.1 mm to (331.9, 123.5), turned to -90 degrees
- moved H2 63.1 mm to (337.4, 185.0), turned to 180 degrees
- moved H1 57.4 mm to (391.9, 186.7), turned to 180 degrees
- moved C5 54.3 mm to (330.9, 147.0), turned to -90 degrees
- moved F1 52.0 mm to (384.2, 186.7), turned to 180 degrees
- moved C4 48.5 mm to (338.4, 137.5), turned to -90 degrees
- moved R2 47.0 mm to (341.6, 172.5), turned to 180 degrees
- moved C6 44.6 mm to (337.9, 147.0), turned to -90 degrees
- moved S1 40.8 mm to (344.2, 168.4), turned to 0 degrees
- moved C2 37.0 mm to (354.4, 131.5), turned to 180 degrees
- moved D1 23.6 mm to (356.0, 164.0), turned to 180 degrees
- moved R1 20.1 mm to (356.5, 160.5), turned to 180 degrees
- moved C1 20.1 mm to (355.6, 148.0), turned to 180 degrees
Routing:
- net +VDC: track 117.0 -> 211.9 mm
- net CSense_OUT_LES: track 2.00 -> 18.2 mm
- net -VDC: track 119.9 -> 128.4 mm

Commit message: update Current sense
Parts:
- removed C42: 10uF, Capacitor_THT:C_Axial_L17.0mm_D7.0mm_P25.00mm_Horizontal
- removed C43: 100nf, Capacitor_THT:C_Disc_D10.5mm_W5.0mm_P5.00mm
- removed C44: 4.7uF, Capacitor_THT:C_Axial_L17.0mm_D7.0mm_P25.00mm_Horizontal
- removed D4, D5, D6: UF4007, Diode_THT:D_DO-35_SOD27_P7.62mm_Horizontal
- removed H3: PHASE_A, MountingHole:MountingHole_3.7mm_Pad_Via
- removed the H4 at (78.8, 89.6)
- removed H5: PHASE_C, MountingHole:MountingHole_3.7mm_Pad_Via
- removed P1: TYPE_C Receptacle, Connector_USB:USB_C_Receptacle_HRO_TYPE-C-31-M-12
- removed Q10, Q11, Q12, Q13, Q2, Q3, Q4, Q5: IXTP90N15T, Package_TO_SOT_THT:SIPAK_Vertical
- removed the Q6 at (53.9, 53.4)
- removed the Q7 at (53.9, 57.3)
- removed the Q8 at (53.9, 61.1)
- removed the Q9 at (53.9, 65.0)
- removed R29, R38, R39, R46, R47, R48, R49: 10K, Resistor_THT:R_Axial_DIN0207_L6.3mm_D2.5mm_P7.62mm_Horizontal
- removed the R30 at (72.6, 37.7)
- removed the R31 at (72.6, 41.8)
- removed the R32 at (72.6, 45.8)
- removed the R33 at (72.6, 49.9)
- removed the R34 at (72.6, 53.9)
- removed the R35 at (72.6, 58.0)
- removed the R36 at (72.6, 62.0)
- removed the R37 at (72.6, 66.1)
- removed R40, R41: 100, Resistor_THT:R_Axial_DIN0207_L6.3mm_D2.5mm_P7.62mm_Horizontal
- removed R42, R43, R44, R45: 22, Resistor_THT:R_Axial_DIN0207_L6.3mm_D2.5mm_P7.62mm_Horizontal
- removed U5, U7: IR2110, Package_DIP:DIP-14_W7.62mm
- added C46: 10uF, Capacitor_SMD:C_0603_1608Metric_Pad1.08x0.95mm_HandSolder, B.Cu at (255.8, 114.8)
- added C47: 100nF, Capacitor_SMD:C_0603_1608Metric_Pad1.08x0.95mm_HandSolder, B.Cu at (254.4, 114.8)
- added C48: 100nF, Capacitor_SMD:C_0603_1608Metric_Pad1.08x0.95mm_HandSolder, F.Cu at (255.6, 121.6)
- added C49: 10uF, Capacitor_SMD:C_0603_1608Metric_Pad1.08x0.95mm_HandSolder, F.Cu at (255.6, 123.1)
- added C50: 100nF, Capacitor_SMD:C_0603_1608Metric_Pad1.08x0.95mm_HandSolder, F.Cu at (255.6, 124.6)
- added C51: 100nF, Capacitor_SMD:C_0603_1608Metric_Pad1.08x0.95mm_HandSolder, F.Cu at (268.1, 122.0)
- added C52: 10uF, Capacitor_SMD:C_0603_1608Metric_Pad1.08x0.95mm_HandSolder, F.Cu at (269.6, 122.0)
- added C53: 100nF, Capacitor_SMD:C_0603_1608Metric_Pad1.08x0.95mm_HandSolder, F.Cu at (271.2, 122.0)
- added C54: 100nF, Capacitor_SMD:C_0603_1608Metric_Pad1.08x0.95mm_HandSolder, F.Cu at (270.8, 105.5)
- added C55: 10uF, Capacitor_SMD:C_0603_1608Metric_Pad1.08x0.95mm_HandSolder, F.Cu at (272.3, 105.5)
- added C56: 100nF, Capacitor_SMD:C_0603_1608Metric_Pad1.08x0.95mm_HandSolder, F.Cu at (273.8, 105.5)
- added C57: 4.7uF, Capacitor_THT:C_Rect_L7.2mm_W3.5mm_P5.00mm_FKS2_FKP2_MKS2_MKP2, F.Cu at (258.1, 159.2)
- added C58: 100uf, Capacitor_SMD:C_0805_2012Metric_Pad1.18x1.45mm_HandSolder, B.Cu at (190.2, 159.8)
- added C59: 100uf, Capacitor_SMD:C_0805_2012Metric_Pad1.18x1.45mm_HandSolder, B.Cu at (226.1, 161.2)
- added C60: 100uf, Capacitor_SMD:C_0805_2012Metric_Pad1.18x1.45mm_HandSolder, B.Cu at (258.0, 161.8)
- added C61: 10uF, Capacitor_SMD:C_1210_3225Metric_Pad1.33x2.70mm_HandSolder, F.Cu at (266.3, 255.7)
- added C62: 10uF, Capacitor_SMD:C_1210_3225Metric_Pad1.33x2.70mm_HandSolder, F.Cu at (266.3, 260.0)
- added C63: 100nF, Capacitor_SMD:C_0805_2012Metric_Pad1.18x1.45mm_HandSolder, F.Cu at (265.7, 219.3)
- added C64: 100nF, Capacitor_SMD:C_0805_2012Metric_Pad1.18x1.45mm_HandSolder, F.Cu at (265.7, 222.3)
- added C65: 100nF, Capacitor_SMD:C_0805_2012Metric_Pad1.18x1.45mm_HandSolder, F.Cu at (265.7, 225.3)
- added C66: 100nF, Capacitor_SMD:C_0805_2012Metric_Pad1.18x1.45mm_HandSolder, F.Cu at (265.7, 228.3)
- added C67: 100nF, Capacitor_SMD:C_0805_2012Metric_Pad1.18x1.45mm_HandSolder, F.Cu at (265.7, 231.3)
- added C68: 10uF, Capacitor_SMD:C_1210_3225Metric_Pad1.33x2.70mm_HandSolder, F.Cu at (240.1, 255.7)
- added C69: 10uF, Capacitor_SMD:C_1210_3225Metric_Pad1.33x2.70mm_HandSolder, F.Cu at (240.1, 260.0)
- added C70: 100nF, Capacitor_SMD:C_0805_2012Metric_Pad1.18x1.45mm_HandSolder, F.Cu at (239.5, 219.3)
- added C71: 100nF, Capacitor_SMD:C_0805_2012Metric_Pad1.18x1.45mm_HandSolder, F.Cu at (239.5, 222.3)
- added C72: 100nF, Capacitor_SMD:C_0805_2012Metric_Pad1.18x1.45mm_HandSolder, F.Cu at (239.5, 225.3)
- added C73: 100nF, Capacitor_SMD:C_0805_2012Metric_Pad1.18x1.45mm_HandSolder, F.Cu at (239.5, 228.3)
- added C74: 100nF, Capacitor_SMD:C_0805_2012Metric_Pad1.18x1.45mm_HandSolder, F.Cu at (239.5, 231.3)
- added C75: 10uF, Capacitor_SMD:C_1210_3225Metric_Pad1.33x2.70mm_HandSolder, F.Cu at (213.8, 255.7)
- added C76: 10uF, Capacitor_SMD:C_1210_3225Metric_Pad1.33x2.70mm_HandSolder, F.Cu at (213.8, 260.0)
- added C77: 100nF, Capacitor_SMD:C_0805_2012Metric_Pad1.18x1.45mm_HandSolder, F.Cu at (213.2, 219.3)
- added C78: 100nF, Capacitor_SMD:C_0805_2012Metric_Pad1.18x1.45mm_HandSolder, F.Cu at (213.2, 222.3)
- added C79: 100nF, Capacitor_SMD:C_0805_2012Metric_Pad1.18x1.45mm_HandSolder, F.Cu at (213.2, 225.3)
- added C80: 100nF, Capacitor_SMD:C_0805_2012Metric_Pad1.18x1.45mm_HandSolder, F.Cu at (213.2, 228.3)
- added C81: 100nF, Capacitor_SMD:C_0805_2012Metric_Pad1.18x1.45mm_HandSolder, F.Cu at (213.2, 231.3)
- added H4: PHASE_B, MountingHole:MountingHole_3.7mm_Pad_Via, F.Cu at (229.0, 192.8)
- added H4: PHASE_B, MountingHole:MountingHole_3.7mm_Pad_Via, F.Cu at (241.5, 249.1)
- added H6: PHASE_A, MountingHole:MountingHole_3.7mm_Pad_Via, F.Cu at (263.5, 193.1)
- added H6: PHASE_A, MountingHole:MountingHole_3.7mm_Pad_Via, F.Cu at (267.8, 249.1)
- added H7: PHASE_C, MountingHole:MountingHole_3.7mm_Pad_Via, F.Cu at (194.4, 192.0)
- added H7: PHASE_C, MountingHole:MountingHole_3.7mm_Pad_Via, F.Cu at (215.3, 249.1)
- added J11: USB_C_Receptacle, Connector_USB:USB_C_Receptacle_GCT_USB4105-xx-A_16P_TopMnt_Horizontal, F.Cu at (284.2, 110.4)
- added J12: Conn_01x02, Connector_PinSocket_2.00mm:PinSocket_1x02_P2.00mm_Horizontal, F.Cu at (55.3, 74.1)
- added J13: OUTSIDE LED, Connector_PinSocket_2.00mm:PinSocket_1x02_P2.00mm_Horizontal, F.Cu at (55.3, 80.2)
- added JP1: Jumper_3_Open, Connector_PinHeader_1.27mm:PinHeader_1x03_P1.27mm_Horizontal, F.Cu at (59.0, 86.9)
- added NT1: NetTie_2, NetTie:NetTie-2_SMD_Pad2.0mm, B.Cu at (30.7, 69.0)
- added NT2: NetTie_2, NetTie:NetTie-2_SMD_Pad0.5mm, B.Cu at (248.2, 104.8)
- added NT3: NetTie_2, NetTie:NetTie-2_SMD_Pad0.5mm, B.Cu at (255.3, 111.2)
- added NT4: NetTie_2, NetTie:NetTie-2_SMD_Pad0.5mm, F.Cu at (272.0, 121.1)
- added NT5: NetTie_2, NetTie:NetTie-2_SMD_Pad0.5mm, F.Cu at (256.5, 125.4)
- added NT6: NetTie_2, NetTie:NetTie-2_SMD_Pad0.5mm, F.Cu at (251.0, 101.9)
- added NT7: NetTie_2, NetTie:NetTie-2_SMD_Pad0.5mm, F.Cu at (274.5, 104.7)
- added NT9: NetTie_2, NetTie:NetTie-2_SMD_Pad0.5mm, B.Cu at (256.6, 114.0)
- added Q14: IAUS300N08S5N0, MOSFET:TRANS_IAUS300N08S5N014ATMA1, F.Cu at (272.1, 184.1)
- added Q14: IAUS300N08S5N0, MOSFET:TRANS_IAUS300N08S5N014ATMA1, F.Cu at (255.9, 223.6)
- added Q15: IAUS300N08S5N0, MOSFET:TRANS_IAUS300N08S5N014ATMA1, F.Cu at (272.1, 171.3)
- added Q15: IAUS300N08S5N0, MOSFET:TRANS_IAUS300N08S5N014ATMA1, F.Cu at (255.9, 235.3)
- added Q16: IAUS300N08S5N0, MOSFET:TRANS_IAUS300N08S5N014ATMA1, F.Cu at (254.7, 171.4)
- added Q16: IAUS300N08S5N0, MOSFET:TRANS_IAUS300N08S5N014ATMA1, F.Cu at (255.9, 246.9)
- added Q17: IAUS300N08S5N0, MOSFET:TRANS_IAUS300N08S5N014ATMA1, F.Cu at (255.9, 258.6)
- added Q17: IAUS300N08S5N0, MOSFET:TRANS_IAUS300N08S5N014ATMA1, F.Cu at (254.7, 184.1)
- added Q18: IAUS300N08S5N0, MOSFET:TRANS_IAUS300N08S5N014ATMA1, F.Cu at (203.4, 223.6)
- added Q18: IAUS300N08S5N0, MOSFET:TRANS_IAUS300N08S5N014ATMA1, F.Cu at (203.5, 170.6)
- added Q19: IAUS300N08S5N0, MOSFET:TRANS_IAUS300N08S5N014ATMA1, F.Cu at (186.1, 170.1)
- added Q19: IAUS300N08S5N0, MOSFET:TRANS_IAUS300N08S5N014ATMA1, F.Cu at (203.4, 235.3)
- added Q20: IAUS300N08S5N0, MOSFET:TRANS_IAUS300N08S5N014ATMA1, F.Cu at (203.4, 183.5)
- added Q20: IAUS300N08S5N0, MOSFET:TRANS_IAUS300N08S5N014ATMA1, F.Cu at (203.4, 246.9)
- added Q21: IAUS300N08S5N0, MOSFET:TRANS_IAUS300N08S5N014ATMA1, F.Cu at (185.9, 182.8)
- added Q21: IAUS300N08S5N0, MOSFET:TRANS_IAUS300N08S5N014ATMA1, F.Cu at (203.4, 258.6)
- added Q6: IAUS300N08S5N0, MOSFET:TRANS_IAUS300N08S5N014ATMA1, F.Cu at (237.7, 170.9)
- added Q6: IAUS300N08S5N0, MOSFET:TRANS_IAUS300N08S5N014ATMA1, F.Cu at (229.7, 223.6)
- added Q7: IAUS300N08S5N0, MOSFET:TRANS_IAUS300N08S5N014ATMA1, F.Cu at (229.7, 235.3)
- added Q7: IAUS300N08S5N0, MOSFET:TRANS_IAUS300N08S5N014ATMA1, F.Cu at (219.9, 183.5)
- added Q8: IAUS300N08S5N0, MOSFET:TRANS_IAUS300N08S5N014ATMA1, F.Cu at (237.6, 183.7)
- added Q8: IAUS300N08S5N0, MOSFET:TRANS_IAUS300N08S5N014ATMA1, F.Cu at (229.7, 246.9)
- added Q9: IAUS300N08S5N0, MOSFET:TRANS_IAUS300N08S5N014ATMA1, F.Cu at (229.7, 258.6)
- added Q9: IAUS300N08S5N0, MOSFET:TRANS_IAUS300N08S5N014ATMA1, F.Cu at (219.9, 170.7)
- added R13: 10R, Resistor_SMD:R_0805_2012Metric_Pad1.20x1.40mm_HandSolder, F.Cu at (265.7, 234.3)
- added R13: 10R, Resistor_SMD:R_0805_2012Metric_Pad1.20x1.40mm_HandSolder, F.Cu at (266.1, 177.8)
- added R30: 10R, Resistor_SMD:R_0805_2012Metric_Pad1.20x1.40mm_HandSolder, F.Cu at (232.2, 164.1)
- added R30: 10R, Resistor_SMD:R_0805_2012Metric_Pad1.20x1.40mm_HandSolder, F.Cu at (239.4, 234.3)
- added R31: 10R, Resistor_SMD:R_0805_2012Metric_Pad1.20x1.40mm_HandSolder, F.Cu at (213.5, 177.2)
- added R31: 10R, Resistor_SMD:R_0805_2012Metric_Pad1.20x1.40mm_HandSolder, F.Cu at (239.4, 237.3)
- added R32: 10R, Resistor_SMD:R_0805_2012Metric_Pad1.20x1.40mm_HandSolder, F.Cu at (239.4, 240.2)
- added R32: 10R, Resistor_SMD:R_0805_2012Metric_Pad1.20x1.40mm_HandSolder, F.Cu at (231.9, 177.4)
- added R33: 10R, Resistor_SMD:R_0805_2012Metric_Pad1.20x1.40mm_HandSolder, F.Cu at (239.4, 243.2)
- added R33: 10R, Resistor_SMD:R_0805_2012Metric_Pad1.20x1.40mm_HandSolder, F.Cu at (213.6, 164.3)
- added R34: 10R, Resistor_SMD:R_0805_2012Metric_Pad1.20x1.40mm_HandSolder, F.Cu at (197.1, 164.3)
- added R34: 10R, Resistor_SMD:R_0805_2012Metric_Pad1.20x1.40mm_HandSolder, F.Cu at (213.2, 234.3)
- added R35: 10R, Resistor_SMD:R_0805_2012Metric_Pad1.20x1.40mm_HandSolder, F.Cu at (180.2, 163.8)
- added R35: 10R, Resistor_SMD:R_0805_2012Metric_Pad1.20x1.40mm_HandSolder, F.Cu at (213.2, 237.3)
- added R36: 10R, Resistor_SMD:R_0805_2012Metric_Pad1.20x1.40mm_HandSolder, F.Cu at (197.7, 177.2)
- added R36: 10R, Resistor_SMD:R_0805_2012Metric_Pad1.20x1.40mm_HandSolder, F.Cu at (213.2, 240.2)
- added R37: 10R, Resistor_SMD:R_0805_2012Metric_Pad1.20x1.40mm_HandSolder, F.Cu at (213.2, 243.2)
- added R37: 10R, Resistor_SMD:R_0805_2012Metric_Pad1.20x1.40mm_HandSolder, F.Cu at (180.0, 176.5)
- added R55: 10R, Resistor_SMD:R_0805_2012Metric_Pad1.20x1.40mm_HandSolder, F.Cu at (266.3, 165.3)
- added R55: 10R, Resistor_SMD:R_0805_2012Metric_Pad1.20x1.40mm_HandSolder, F.Cu at (265.7, 237.3)
- added R56: 10R, Resistor_SMD:R_0805_2012Metric_Pad1.20x1.40mm_HandSolder, F.Cu at (248.4, 165.1)
- added R56: 10R, Resistor_SMD:R_0805_2012Metric_Pad1.20x1.40mm_HandSolder, F.Cu at (265.7, 240.2)
- added R57: 10R, Resistor_SMD:R_0805_2012Metric_Pad1.20x1.40mm_HandSolder, F.Cu at (265.7, 243.2)
- added R57: 10R, Resistor_SMD:R_0805_2012Metric_Pad1.20x1.40mm_HandSolder, F.Cu at (248.7, 177.8)
- added U10: IRS21867S, Package_SO:SOIC-8_3.9x4.9mm_P1.27mm, F.Cu at (195.1, 156.1)
- added U12: TMP101, Package_TO_SOT_SMD:SOT-23-6, F.Cu at (266.1, 99.0)
- added U9: IRS21867S, Package_SO:SOIC-8_3.9x4.9mm_P1.27mm, F.Cu at (264.0, 156.8)
- C1, C2, C3: footprint Capacitor_THT:C_Radial_D16.0mm_H31.5mm_P7.50mm -> Capacitor_THT:CP_Radial_D18.0mm_P7.50mm
- C18, C20, C21, C23, C24, J1: moved to B.Cu
- C19, C22: value 100nF -> 10uF; moved to B.Cu
- C33, C34, C35: footprint Capacitor_THT:C_Disc_D10.5mm_W5.0mm_P5.00mm -> Capacitor_SMD:C_0603_1608Metric_Pad1.08x0.95mm_HandSolder
- C36: value 100nf -> 100nF; footprint Capacitor_THT:C_Disc_D10.5mm_W5.0mm_P5.00mm -> Capacitor_SMD:C_0603_1608Metric_Pad1.08x0.95mm_HandSolder
- C37, C41: value 4.7uF -> 100nF; footprint Capacitor_THT:C_Axial_L17.0mm_D7.0mm_P25.00mm_Horizontal -> Capacitor_SMD:C_0603_1608Metric_Pad1.08x0.95mm_HandSolder
- C38: footprint Capacitor_THT:C_Radial_D12.5mm_H25.0mm_P5.00mm -> Capacitor_SMD:C_0603_1608Metric_Pad1.08x0.95mm_HandSolder
- C39: value 10uF -> 4.7uF; footprint Capacitor_THT:C_Radial_D12.5mm_H25.0mm_P5.00mm -> Capacitor_THT:C_Rect_L7.2mm_W3.5mm_P5.00mm_FKS2_FKP2_MKS2_MKP2
- C4, C5, C6: footprint Capacitor_THT:C_Radial_D6.3mm_H11.0mm_P2.50mm -> Capacitor_SMD:C_1210_3225Metric_Pad1.33x2.70mm_HandSolder
- C40: value 100nf -> 4.7uF; footprint Capacitor_THT:C_Disc_D10.5mm_W5.0mm_P5.00mm -> Capacitor_THT:C_Rect_L7.2mm_W3.5mm_P5.00mm_FKS2_FKP2_MKS2_MKP2
- C45: value C -> 100nF
- R10, R14, R15, R16, R17, R18, R19, R51, R52, R53, R54, R9: footprint Resistor_THT:R_Axial_DIN0207_L6.3mm_D2.5mm_P7.62mm_Horizontal -> Resistor_SMD:R_0603_1608Metric_Pad0.98x0.95mm_HandSolder
- R20: value 22 -> 4.7K
- R21: value 22 -> 260; footprint Resistor_THT:R_Axial_DIN0207_L6.3mm_D2.5mm_P7.62mm_Horizontal -> Resistor_SMD:R_0603_1608Metric_Pad0.98x0.95mm_HandSolder
- R22: value 22 -> 120R; footprint Resistor_THT:R_Axial_DIN0207_L6.3mm_D2.5mm_P7.62mm_Horizontal -> Resistor_SMD:R_0603_1608Metric_Pad0.98x0.95mm_HandSolder
- R23: value 22 -> 100; footprint Resistor_THT:R_Axial_DIN0207_L6.3mm_D2.5mm_P7.62mm_Horizontal -> Resistor_SMD:R_0603_1608Metric_Pad0.98x0.95mm_HandSolder
- R24, R25: value 100 -> 4.7K; footprint Resistor_THT:R_Axial_DIN0207_L6.3mm_D2.5mm_P7.62mm_Horizontal -> Resistor_SMD:R_0603_1608Metric_Pad0.98x0.95mm_HandSolder
- R26, R27, R28: value 10K -> 10R; footprint Resistor_THT:R_Axial_DIN0207_L6.3mm_D2.5mm_P7.62mm_Horizontal -> Resistor_SMD:R_0805_2012Metric_Pad1.20x1.40mm_HandSolder
- R4: value 88.7K -> 86.6K
- R6: value 147K -> 46k
- R8: footprint Resistor_THT:R_Axial_DIN0207_L6.3mm_D2.5mm_P7.62mm_Horizontal -> Resistor_SMD:R_0402_1005Metric_Pad0.72x0.64mm_HandSolder
- U6: value IR2110 -> IRS21867S; footprint Package_DIP:DIP-14_W7.62mm -> Package_SO:SOIC-8_3.9x4.9mm_P1.27mm
- moved R12 330.8 mm to (37.5, 60.0)
- moved R11 328.7 mm to (37.5, 56.0), turned to 0 degrees
- moved D3 323.7 mm to (52.4, 86.2), turned to 0 degrees
- moved Q1 311.2 mm to (53.1, 90.5), turned to 0 degrees
- moved R2 291.4 mm to (81.2, 41.8), turned to 0 degrees
- moved F1 260.9 mm to (200.0, 1.85), turned to -90 degrees
- moved H1 259.4 mm to (207.5, 4.25), turned to -90 degrees
- moved C8 238.2 mm to (96.1, 91.0), turned to 0 degrees
- moved D2 237.0 mm to (125.1, 23.9), turned to 0 degrees
- moved R1 232.9 mm to (198.4, -10.6), turned to 0 degrees
- moved C7 227.8 mm to (159.7, 22.6), turned to 0 degrees
- moved D1 226.0 mm to (207.5, -6.45), turned to 0 degrees
- moved R26 225.3 mm to (263.1, 163.3), turned to -90 degrees
- moved R24 212.1 mm to (269.2, 98.9), turned to -90 degrees
- moved R23 209.5 mm to (266.6, 94.5), turned to -90 degrees
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Connections:
- net USB_DM renamed D-
- net USB_DP renamed D+
- BZ1 pad 1: Net-(BZ1-+) -> +5V
- C18 pad 2: +3V3 -> VBAT
- C19 pad 2: +3V3 -> VBAT
- C20 pad 2: +3V3 -> VBAT
- C21 pad 2: +3V3 -> VDD_1
- C22 pad 2: +3V3 -> VDD_1
- C23 pad 2: +3V3 -> VDD_1
- C24 pad 2: +3V3 -> VDD_2
- C36 pad 1: +12V -> Net-(U8-VIQ)
- C36 pad 2: -VDC -> GND
- C37 pad 1: Net-(D4-A) -> GND
- C37 pad 2: +12V -> VDD_6
- C38 pad 1: +12V -> GND
- C38 pad 2: -VDC -> VDD_6
- C39 pad 1: +12V -> Net-(U6-VB)
- C39 pad 2: -VDC -> Phase_B
- C40 pad 1: +12V -> Net-(U10-VB)
- C40 pad 2: -VDC -> Phase_C
- C41 pad 1: Net-(D5-A) -> GND
- C41 pad 2: +12V -> VDD_6
- D2 pad 1: Net-(BZ1-+) -> +5V
- D2 pad 2: +5V -> Net-(BZ1--)
- R12 pad 1: STATUS_LED -> Net-(JP1-C)
- R12 pad 2: Net-(D3-A) -> Net-(J13-Pin_2)
- R20 pad 1: Net-(U5-LO) -> Net-(Q1-B)
- R20 pad 2: Net-(Q3-G) -> GND
- R21 pad 1: Net-(U5-LO) -> Net-(JP1-B)
- R21 pad 2: Net-(Q5-G) -> Net-(D3-A)
- R22 pad 1: Net-(U5-HO) -> Net-(J3-Pin_2)
- R22 pad 2: Net-(Q4-G) -> Net-(J3-Pin_1)
- R23 pad 1: Net-(U5-HO) -> +3V3
- R23 pad 2: Net-(Q2-G) -> TMP_ALERT
- R24 pad 1: HS_MOS_A -> +3V3
- R24 pad 2: Net-(U5-HIN) -> TMP_SCL
- R25 pad 1: Net-(U5-LIN) -> +3V3
- R25 pad 2: LS_MOS_A -> TMP_SDA
- R26 pad 1: Net-(Q4-G) -> Net-(U9-VS)
- R26 pad 2: Net-(Q2-S) -> Phase_A
- R27 pad 1: Net-(Q2-G) -> Net-(U6-VS)
- R27 pad 2: Net-(Q2-S) -> Phase_B
- R28 pad 1: -VDC -> Net-(U10-VS)
- R28 pad 2: Net-(Q3-G) -> Phase_C
- U1 pad 100: +3V3 -> VDD_6
- U1 pad 11: +3V3 -> VDD_1
- U1 pad 19: +3V3 -> VDD_2
- U1 pad 28: +3V3 -> VDD_3
- U1 pad 43: HS_MOS_C -> LS_MOS_C
- U1 pad 47: BT_TX -> CAN_S
- U1 pad 48: BT_RX -> BT_TX
- U1 pad 50: +3V3 -> VDD_4
- U1 pad 51: BT_KEY -> BT_RX
- U1 pad 52: unconnected-(U1-PB13-Pad52) -> BT_KEY
- U1 pad 6: +3V3 -> VBAT
- U1 pad 75: +3V3 -> VDD_5
- U1 pad 81: unconnected-(U1-PD0-Pad81) -> TMP_SCL
- U1 pad 82: unconnected-(U1-PD1-Pad82) -> TMP_SDA
- U1 pad 83: unconnected-(U1-PD2-Pad83) -> TMP_ALERT
- U6 pad 1: Net-(U6-LO) -> +12V
- U6 pad 2: -VDC -> HS_MOS_B
- U6 pad 3: +12V -> LS_MOS_B
- U6 pad 4: unconnected-(U6-NC-Pad4) -> GND
- U6 pad 5: Net-(Q6-S) -> L_MOS_OUT_B
- U6 pad 6: Net-(D5-K) -> Net-(U6-VS)
- U6 pad 7: Net-(U6-HO) -> H_MOS_OUT_B
- U6 pad 8: unconnected-(U6-NC-Pad8) -> Net-(U6-VB)
- U8 pad 5: unconnected-(U8-NC-Pad5) -> Net-(U8-VIQ)
- U8 pad 8: GND -> CAN_S
Routing:
- net +VDC: track 211.9 -> 111.5 mm
- net -VDC: track 128.4 -> 51.2 mm
- net L_MOS_OUT_A: track 0.00 -> 42.4 mm, vias 0 -> 2
- net L_MOS_OUT_B: track 0.00 -> 39.7 mm, vias 0 -> 2
- net L_MOS_OUT_C: track 0.00 -> 38.8 mm, vias 0 -> 2
- net Net-(J2-Pin_3): track 0.00 -> 31.7 mm, vias 0 -> 1
- net GND: track 13.1 -> 43.9 mm, vias 0 -> 5
- net H_MOS_OUT_C: track 0.00 -> 30.2 mm, vias 0 -> 2
- net H_MOS_OUT_A: track 0.00 -> 29.4 mm, vias 0 -> 2
- net H_MOS_OUT_B: track 0.00 -> 27.3 mm, vias 0 -> 2
- net Net-(J2-Pin_2): track 0.00 -> 22.0 mm, vias 0 -> 1
- net CSense_OUT_LES: track 18.2 -> 0.00 mm, vias 1 -> 0
- net STATUS_LED: track 16.2 -> 0.00 mm
- net /MCU/I2C_SCL: track 21.9 -> 6.17 mm
- net SWDIO: track 0.00 -> 15.7 mm
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- added copper zone on F.Cu, net Phase_A
- added copper zone on F.Cu, net Phase_B
- added copper zone on F.Cu, net Phase_C
- removed copper zone on F.Cu, net GND
- removed copper zone on In1.Cu, net GND
Other:
- board text added: "10R"

Commit message: update: revised label
Parts:
- removed the H4 at (229.0, 192.8)
- removed the H4 at (241.5, 249.1)
- removed the H6 at (267.8, 249.1)
- removed the H7 at (194.4, 192.0)
- removed the H7 at (215.3, 249.1)
- removed the Q14 at (255.9, 223.6)
- removed the Q15 at (255.9, 235.3)
- removed the Q16 at (255.9, 246.9)
- removed the Q17 at (255.9, 258.6)
- removed the Q18 at (203.4, 223.6)
- removed the Q18 at (203.5, 170.6)
- removed the Q19 at (186.1, 170.1)
- removed the Q19 at (203.4, 235.3)
- removed the Q20 at (203.4, 183.5)
- removed the Q20 at (203.4, 246.9)
- removed the Q21 at (185.9, 182.8)
- removed the Q21 at (203.4, 258.6)
- removed the Q6 at (237.7, 170.9)
- removed the Q6 at (229.7, 223.6)
- removed the Q7 at (229.7, 235.3)
- removed the Q7 at (219.9, 183.5)
- removed the Q8 at (237.6, 183.7)
- removed the Q8 at (229.7, 246.9)
- removed the Q9 at (229.7, 258.6)
- removed the Q9 at (219.9, 170.7)
- removed the R13 at (265.7, 234.3)
- removed the R30 at (232.2, 164.1)
- removed the R30 at (239.4, 234.3)
- removed the R31 at (213.5, 177.2)
- removed the R31 at (239.4, 237.3)
- removed the R32 at (239.4, 240.2)
- removed the R32 at (231.9, 177.4)
- removed the R33 at (239.4, 243.2)
- removed the R33 at (213.6, 164.3)
- removed the R34 at (197.1, 164.3)
- removed the R34 at (213.2, 234.3)
- removed the R35 at (180.2, 163.8)
- removed the R35 at (213.2, 237.3)
- removed the R36 at (197.7, 177.2)
- removed the R36 at (213.2, 240.2)
- removed the R37 at (213.2, 243.2)
- removed the R37 at (180.0, 176.5)
- removed the R55 at (265.7, 237.3)
- removed the R56 at (265.7, 240.2)
- removed the R57 at (265.7, 243.2)
- added C82: 100nF, Capacitor_SMD:C_0402_1005Metric_Pad0.74x0.62mm_HandSolder, F.Cu at (194.6, 79.9)
- added C83: 10nF, Capacitor_SMD:C_0402_1005Metric_Pad0.74x0.62mm_HandSolder, F.Cu at (191.2, 76.9)
- added C84: 100nF, Capacitor_SMD:C_0402_1005Metric_Pad0.74x0.62mm_HandSolder, F.Cu at (259.1, 88.4)
- added C85: 10nF, Capacitor_SMD:C_0402_1005Metric_Pad0.74x0.62mm_HandSolder, F.Cu at (252.9, 91.1)
- added C86: 100nF, Capacitor_SMD:C_0402_1005Metric_Pad0.74x0.62mm_HandSolder, F.Cu at (148.5, 79.4)
- added C87: 10nF, Capacitor_SMD:C_0402_1005Metric_Pad0.74x0.62mm_HandSolder, F.Cu at (149.4, 83.9)
- added D4: US1M, Diode_SMD:D_SMA, F.Cu at (175.4, 128.2)
- added D5: US1M, Diode_SMD:D_SMA, F.Cu at (222.8, 127.4)
- added D7: US1M, Diode_SMD:D_SMA, F.Cu at (129.2, 127.6)
- added H4: PHASE_B, MountingHole:MountingHole_3.7mm_Pad_Via, F.Cu at (180.8, 91.1)
- added H7: PHASE_C, MountingHole:MountingHole_3.7mm_Pad_Via, F.Cu at (227.9, 90.9)
- added Q18: IAUS300N08S5N0, MOSFET:TRANS_IAUS300N08S5N014ATMA1, F.Cu at (219.2, 99.9)
- added Q19: IAUS300N08S5N0, MOSFET:TRANS_IAUS300N08S5N014ATMA1, F.Cu at (236.7, 99.9)
- added Q20: IAUS300N08S5N0, MOSFET:TRANS_IAUS300N08S5N014ATMA1, F.Cu at (219.2, 112.6)
- added Q21: IAUS300N08S5N0, MOSFET:TRANS_IAUS300N08S5N014ATMA1, F.Cu at (236.7, 112.6)
- added Q6: IAUS300N08S5N0, MOSFET:TRANS_IAUS300N08S5N014ATMA1, F.Cu at (172.2, 100.1)
- added Q7: IAUS300N08S5N0, MOSFET:TRANS_IAUS300N08S5N014ATMA1, F.Cu at (189.6, 112.8)
- added Q8: IAUS300N08S5N0, MOSFET:TRANS_IAUS300N08S5N014ATMA1, F.Cu at (172.2, 112.8)
- added Q9: IAUS300N08S5N0, MOSFET:TRANS_IAUS300N08S5N014ATMA1, F.Cu at (189.6, 100.1)
- added R29: 10, Resistor_SMD:R_0402_1005Metric_Pad0.72x0.64mm_HandSolder, F.Cu at (191.9, 75.3)
- added R30: 10R, Resistor_SMD:R_0805_2012Metric_Pad1.20x1.40mm_HandSolder, F.Cu at (178.2, 106.3)
- added R31: 10R, Resistor_SMD:R_0805_2012Metric_Pad1.20x1.40mm_HandSolder, F.Cu at (195.9, 119.1)
- added R32: 10R, Resistor_SMD:R_0805_2012Metric_Pad1.20x1.40mm_HandSolder, F.Cu at (178.0, 118.8)
- added R33: 10R, Resistor_SMD:R_0805_2012Metric_Pad1.20x1.40mm_HandSolder, F.Cu at (195.7, 106.4)
- added R34: 10R, Resistor_SMD:R_0805_2012Metric_Pad1.20x1.40mm_HandSolder, F.Cu at (225.2, 106.1)
- added R35: 10R, Resistor_SMD:R_0805_2012Metric_Pad1.20x1.40mm_HandSolder, F.Cu at (242.9, 118.9)
- added R36: 10R, Resistor_SMD:R_0805_2012Metric_Pad1.20x1.40mm_HandSolder, F.Cu at (225.0, 118.6)
- added R37: 10R, Resistor_SMD:R_0805_2012Metric_Pad1.20x1.40mm_HandSolder, F.Cu at (242.7, 106.2)
- added R38: 1mR, Resistor_SMD:R_2512_6332Metric_Pad1.40x3.35mm_HandSolder, B.Cu at (191.0, 75.4)
- added R39: 10, Resistor_SMD:R_0402_1005Metric_Pad0.72x0.64mm_HandSolder, F.Cu at (190.7, 75.3)
- added R58: 10k, Resistor_SMD:R_1812_4532Metric_Pad1.30x3.40mm_HandSolder, F.Cu at (202.1, 80.7)
- added R59: 10k, Resistor_SMD:R_1812_4532Metric_Pad1.30x3.40mm_HandSolder, F.Cu at (202.1, 76.2)
- added R60: 10, Resistor_SMD:R_0402_1005Metric_Pad0.72x0.64mm_HandSolder, F.Cu at (251.9, 89.0)
- added R61: 1mR, Resistor_SMD:R_2512_6332Metric_Pad1.40x3.35mm_HandSolder, B.Cu at (251.1, 90.9)
- added R62: 10, Resistor_SMD:R_0402_1005Metric_Pad0.72x0.64mm_HandSolder, F.Cu at (251.8, 92.1)
- added R63: 10k, Resistor_SMD:R_1812_4532Metric_Pad1.30x3.40mm_HandSolder, F.Cu at (256.0, 85.6)
- added R64: 10k, Resistor_SMD:R_1812_4532Metric_Pad1.30x3.40mm_HandSolder, F.Cu at (262.6, 85.6)
- added R65: 10, Resistor_SMD:R_0402_1005Metric_Pad0.72x0.64mm_HandSolder, F.Cu at (147.5, 83.5)
- added R66: 1mR, Resistor_SMD:R_2512_6332Metric_Pad1.40x3.35mm_HandSolder, B.Cu at (146.4, 86.0)
- added R67: 10, Resistor_SMD:R_0402_1005Metric_Pad0.72x0.64mm_HandSolder, F.Cu at (149.8, 85.9)
- added R68: 10k, Resistor_SMD:R_1812_4532Metric_Pad1.30x3.40mm_HandSolder, F.Cu at (142.6, 83.6)
- added R69: 10k, Resistor_SMD:R_1812_4532Metric_Pad1.30x3.40mm_HandSolder, F.Cu at (142.6, 77.2)
- added U11: INA241A2, Package_TO_SOT_SMD:SOT-23-8_Handsoldering, F.Cu at (255.2, 90.8)
- added U13: INA241A2, Package_TO_SOT_SMD:SOT-23-8_Handsoldering, F.Cu at (151.0, 82.4)
- added U5: INA241A2, Package_TO_SOT_SMD:SOT-23-8_Handsoldering, F.Cu at (191.4, 79.0)
- C40, C61, C62, C63, C64, C65, C66, C67, C68, C69, C70, C71, C72, C73, C74, C75, C76, C77, C78, C79, C80, C81: moved to B.Cu
- moved BZ1 270.6 mm to (1.57, 85.2), turned to 90 degrees
- moved J9 258.2 mm to (-7.75, 109.6), turned to -90 degrees
- moved J11 256.1 mm to (30.8, 73.1), turned to 180 degrees
- moved J5 253.1 mm to (18.2, 86.3), turned to 180 degrees
- moved R23 251.7 mm to (14.9, 90.8), turned to 0 degrees
- moved R52 250.9 mm to (28.6, 79.5), turned to 90 degrees
- moved NT7 250.3 mm to (25.1, 82.8), turned to 90 degrees
- moved R24 250.1 mm to (19.3, 88.1), turned to 0 degrees
- moved R54 249.5 mm to (30.1, 79.6), turned to 90 degrees
- moved J8 249.2 mm to (0.30, 109.6), turned to -90 degrees
- moved C56 248.8 mm to (25.9, 83.5), turned to 180 degrees
- moved R53 248.2 mm to (31.6, 79.5), turned to 90 degrees
- moved J2 247.3 mm to (40.5, 73.9), turned to 90 degrees
- moved C55 247.2 mm to (25.9, 85.0), turned to 180 degrees
- moved R51 246.9 mm to (33.1, 79.6), turned to 90 degrees
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Connections:
- net HS_MOS_A renamed /FET/HS_MOS_A
- net H_MOS_OUT_A renamed /FET/H_MOS_OUT_A
- net LS_MOS_A renamed /FET/LS_MOS_A
- net L_MOS_OUT_A renamed /FET/L_MOS_OUT_A
- net Phase_B renamed /FET/Phase_B_FET/PHASE_B
- net Phase_C renamed /FET/Phase_C_FET/PHASE_C
- C57 pad 2: Phase_A -> /FET/Phase_A_FET/PHASE_A
- C60 pad 2: Phase_A -> /FET/Phase_A_FET/PHASE_A
- H6 pad 1: Net-(C57-Pad2) -> /FET/Phase_A_FET/PHASE_A
- Q14 pad 2: Net-(C57-Pad2) -> /FET/Phase_A_FET/PHASE_A
- Q14 pad 3: Net-(C57-Pad2) -> /FET/Phase_A_FET/PHASE_A
- Q14 pad 4: Net-(C57-Pad2) -> /FET/Phase_A_FET/PHASE_A
- Q14 pad 5: Net-(C57-Pad2) -> /FET/Phase_A_FET/PHASE_A
- Q14 pad 6: Net-(C57-Pad2) -> /FET/Phase_A_FET/PHASE_A
- Q14 pad 7: Net-(C57-Pad2) -> /FET/Phase_A_FET/PHASE_A
- Q14 pad 8: Net-(C57-Pad2) -> /FET/Phase_A_FET/PHASE_A
- Q15 pad 2: Net-(C57-Pad2) -> /FET/Phase_A_FET/PHASE_A
- Q15 pad 3: Net-(C57-Pad2) -> /FET/Phase_A_FET/PHASE_A
- Q15 pad 4: Net-(C57-Pad2) -> /FET/Phase_A_FET/PHASE_A
- Q15 pad 5: Net-(C57-Pad2) -> /FET/Phase_A_FET/PHASE_A
- Q15 pad 6: Net-(C57-Pad2) -> /FET/Phase_A_FET/PHASE_A
- Q15 pad 7: Net-(C57-Pad2) -> /FET/Phase_A_FET/PHASE_A
- Q15 pad 8: Net-(C57-Pad2) -> /FET/Phase_A_FET/PHASE_A
- Q16 pad 9: Net-(C57-Pad2) -> /FET/Phase_A_FET/PHASE_A
- Q17 pad 9: Net-(C57-Pad2) -> /FET/Phase_A_FET/PHASE_A
- R26 pad 2: Phase_A -> /FET/Phase_A_FET/PHASE_A
- U1 pad 31: unconnected-(U1-PA6-Pad31) -> Current_Sense_A
- U1 pad 32: unconnected-(U1-PA7-Pad32) -> Current_Sense_B
- U1 pad 35: unconnected-(U1-PB0-Pad35) -> Current_Sense_C
- U1 pad 41: LS_MOS_B -> /FET/HS_MOS_B
- U1 pad 42: HS_MOS_B -> /FET/LS_MOS_B
- U1 pad 43: LS_MOS_C -> HS_MOS_C
- U1 pad 44: HS_MOS_C -> LS_MOS_C
- U10 pad 5: L_MOS_OUT_C -> /FET/L_MOS_OUT_C
- U10 pad 7: H_MOS_OUT_C -> /FET/H_MOS_OUT_C
- U6 pad 2: HS_MOS_B -> /FET/HS_MOS_B
- U6 pad 3: LS_MOS_B -> /FET/LS_MOS_B
- U6 pad 5: L_MOS_OUT_B -> /FET/L_MOS_OUT_B
- U6 pad 7: H_MOS_OUT_B -> /FET/H_MOS_OUT_B
Routing:
- net -VDC: track 51.2 -> 590.6 mm, vias 0 -> 555
- net +VDC: track 111.5 -> 408.5 mm, vias 0 -> 117
- net +3V3: track 15.1 -> 60.7 mm
- net /FET/L_MOS_OUT_C: track 0.00 -> 41.3 mm, vias 0 -> 2
- net /FET/L_MOS_OUT_B: track 0.00 -> 41.3 mm, vias 0 -> 2
- net L_MOS_OUT_B: track 39.7 -> 0.00 mm, vias 2 -> 0
- net L_MOS_OUT_C: track 38.8 -> 0.00 mm, vias 2 -> 0
- net H_MOS_OUT_C: track 30.2 -> 0.00 mm, vias 2 -> 0
- net /FET/H_MOS_OUT_B: track 0.00 -> 29.4 mm, vias 0 -> 2
- net /FET/H_MOS_OUT_C: track 0.00 -> 29.4 mm, vias 0 -> 2
- net H_MOS_OUT_B: track 27.3 -> 0.00 mm, vias 2 -> 0
- net GND: track 43.9 -> 63.7 mm
- net Net-(U5-REF1): track 0.00 -> 11.5 mm
- net Net-(U11-REF1): track 0.00 -> 11.4 mm
- net Net-(U13-REF1): track 0.00 -> 9.84 mm
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- added copper zone on F.Cu, net /FET/Phase_A_FET/PHASE_A
- removed copper zone on F.Cu, net /FET/Phase_C_FET/PHASE_C
- removed copper zone on F.Cu, net Phase_A

Commit message: changes to pcb and footprints
Parts:
- removed F1: Fuse, Fuse:Fuseholder_Littelfuse_445_030_series_5x30mm
- C1, C2, C3: footprint Capacitor_THT:CP_Radial_D18.0mm_P7.50mm -> Capacitor_THT:C_Radial_D16.0mm_H31.5mm_P7.50mm
- C10, C11, C12, C13, C14, C15, C16: footprint Capacitor_THT:C_Disc_D10.5mm_W5.0mm_P10.00mm -> Capacitor_SMD:C_0603_1608Metric_Pad1.08x0.95mm_HandSolder
- C17, C9: footprint Capacitor_THT:C_Disc_D10.5mm_W5.0mm_P10.00mm -> Capacitor_SMD:C_1210_3225Metric_Pad1.33x2.70mm_HandSolder
- C4, C5, C6: footprint Capacitor_SMD:C_1210_3225Metric_Pad1.33x2.70mm_HandSolder -> Capacitor_THT:C_Radial_D6.3mm_H11.0mm_P2.50mm
- L1: footprint Inductor_THT:L_Radial_D10.0mm_P5.00mm_Fastron_07P -> Inductor_SMD:L_1210_3225Metric_Pad1.42x2.65mm_HandSolder
- R3, R4, R5, R6: footprint Resistor_THT:R_Axial_DIN0207_L6.3mm_D2.5mm_P10.16mm_Horizontal -> Resistor_SMD:R_0603_1608Metric_Pad0.98x0.95mm_HandSolder
- moved H1 262.0 mm to (86.5, 57.2), turned to 0 degrees
- moved U3 261.8 mm to (99.8, 160.6), turned to 180 degrees
- moved R2 255.6 mm to (229.5, 175.9)
- moved C14 245.9 mm to (144.5, 206.9)
- moved D2 243.1 mm to (176.6, 162.9)
- moved C7 243.1 mm to (211.2, 161.6)
- moved C36 239.9 mm to (207.8, 209.4)
- moved C45 239.9 mm to (153.0, 165.6)
- moved D3 239.9 mm to (200.7, 203.4)
- moved J10 239.9 mm to (203.6, 185.2)
- moved J13 239.9 mm to (203.6, 197.3)
- moved J3 239.9 mm to (203.6, 173.1)
- moved J4 239.9 mm to (197.0, 203.4)
- moved NT1 239.9 mm to (179.0, 186.1)
- moved Q1 239.9 mm to (201.4, 207.6)
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Connections:
- C9 pad 2: GND -> -VDC
- H1 pad 1: Net-(F1-Pad1) -> Net-(H1-Pad1)
- S1 pad 1: Net-(F1-Pad2) -> Net-(H1-Pad1)
- S1 pad 2: Net-(F1-Pad2) -> Net-(H1-Pad1)
- S1 pad 3: Net-(F1-Pad2) -> Net-(H1-Pad1)
Routing:
- net -VDC: track 590.6 -> 945.7 mm, vias 555 -> 556
- net +VDC: track 408.5 -> 632.7 mm, vias 117 -> 167
- net +12V: track 9.03 -> 213.4 mm
- net Net-(F1-Pad2): track 40.3 -> 0.00 mm
- net ACCEL: track 0.00 -> 36.6 mm, vias 0 -> 1
- net Net-(H1-Pad1): track 0.00 -> 35.0 mm
- net REGEN: track 2.66 -> 31.8 mm
- net Net-(F1-Pad1): track 22.4 -> 0.00 mm
- net Net-(U2-SW): track 0.00 -> 11.6 mm
- net GND: track 63.7 -> 74.8 mm, vias 5 -> 11
- net Net-(U2-FB): track 0.00 -> 7.03 mm
- net Net-(U2-VCC): track 0.00 -> 6.97 mm, vias 0 -> 2
- net Net-(U2-BST): track 0.00 -> 6.46 mm, vias 0 -> 2
- net Net-(C15-Pad1): track 0.00 -> 5.79 mm
- net Net-(U2-RON): track 0.00 -> 1.98 mm
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- added copper zone on F.Cu, net +3V3
- added copper zone on In1.Cu, net GND
Other:
- board outline added: 207.2 x 164.4 mm
