File: Motor_Driver_Shell_Eco.kicad_pcb (KiCad board)
At the start: 6 copper layers, 207.2 x 164.4 mm, 208 parts, among them J1 I2C EKRAN, J10 Conn_01x02, J11 USB_C_Receptacle, J12 Conn_01x02, J13 OUTSIDE LED, J2 HALL INPUT, J3 Conn_01x02, J4 Conn_01x02, J5 Conn_01x04, J6 Conn_01x06, J7 Conn_01x02, J8 Conn_01x03, J9 Conn_01x03, Q1 BC817, Q14 IAUS300N08S5N0, Q15 IAUS300N08S5N0, Q16 IAUS300N08S5N0, Q17 IAUS300N08S5N0, Q18 IAUS300N08S5N0, Q19 IAUS300N08S5N0, Q20 IAUS300N08S5N0, Q21 IAUS300N08S5N0, Q6 IAUS300N08S5N0, Q7 IAUS300N08S5N0, Q8 IAUS300N08S5N0, Q9 IAUS300N08S5N0, SW1 SW_Push, SW2 SW_Push, U1 STM32F205VGTx, U10 IRS21867S, U11 INA241A2, U12 TMP101, U13 INA241A2, U2 LM5017MR, U3 AP2204K-5.0, U4 XC6206 - 3V3, U5 INA241A2, U6 IRS21867S, U8 TJA1051T, U9 IRS21867S, Y1 8MHz

Commit message: LAST I HOPE
Parts:
- added C88: 4.7uF, Capacitor_THT:C_Rect_L7.2mm_W3.5mm_P5.00mm_FKS2_FKP2_MKS2_MKP2, F.Cu at (158.9, 119.0)
- added C89: 100nF, Capacitor_THT:C_Rect_L7.2mm_W3.5mm_P5.00mm_FKS2_FKP2_MKS2_MKP2, F.Cu at (159.5, 169.8)
- added C90: 4.7uF, Capacitor_THT:C_Rect_L7.2mm_W3.5mm_P5.00mm_FKS2_FKP2_MKS2_MKP2, F.Cu at (157.2, 70.0)
- added R70: 1mR, Resistor_SMD:R_2512_6332Metric_Pad1.40x3.35mm_HandSolder, B.Cu at (197.1, 78.2)
- added R71: 1mR, Resistor_SMD:R_2512_6332Metric_Pad1.40x3.35mm_HandSolder, B.Cu at (197.5, 129.0)
- added R72: 1mR, Resistor_SMD:R_2512_6332Metric_Pad1.40x3.35mm_HandSolder, B.Cu at (196.4, 27.4)
- C40, NT1: moved to F.Cu
- C45: footprint Capacitor_THT:C_Axial_L17.0mm_D7.0mm_P25.00mm_Horizontal -> Capacitor_SMD:C_1210_3225Metric_Pad1.33x2.70mm_HandSolder
- D4, D5, D7: moved to B.Cu
- R58, R59, R63, R64, R68, R69: footprint Resistor_SMD:R_1812_4532Metric_Pad1.30x3.40mm_HandSolder -> Resistor_SMD:R_0603_1608Metric_Pad0.98x0.95mm_HandSolder
- moved D1 187.3 mm to (114.3, 51.3), turned to 90 degrees
- moved R1 171.5 mm to (119.0, 56.5), turned to 90 degrees
- moved R2 169.9 mm to (106.2, 59.0), turned to -90 degrees
- moved C7 147.4 mm to (99.0, 66.0), turned to 90 degrees
- moved C8 141.8 mm to (90.6, 66.8), turned to 90 degrees
- moved J10 128.3 mm to (95.9, 115.5)
- moved J12 128.3 mm to (95.9, 121.5)
- moved J13 128.3 mm to (95.9, 127.6)
- moved J7 128.3 mm to (95.9, 109.4)
- moved JP1 127.0 mm to (106.4, 126.8), turned to 90 degrees
- moved D3 125.9 mm to (101.0, 126.5)
- moved C75 116.8 mm to (180.3, 32.2)
- moved C76 116.7 mm to (176.0, 32.2)
- moved C77 115.9 mm to (173.3, 32.8)
- moved C78 115.9 mm to (170.3, 32.8)
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Connections:
- U1 pad 31: Current_Sense_A -> Current Sense_A
- U1 pad 32: Current_Sense_B -> Current Sense_B
- U1 pad 46: unconnected-(U1-PE15-Pad46) -> PANIC STOP
- U1 pad 67: unconnected-(U1-PA8-Pad67) -> Current Sense_C
Routing:
- net -VDC: track 945.7 -> 115.5 mm, vias 556 -> 648
- net +VDC: track 632.7 -> 22.7 mm, vias 167 -> 828
- net GND: track 74.8 -> 465.3 mm, vias 11 -> 29
- net +5V: track 1.15 -> 211.2 mm, vias 0 -> 2
- net Current Sense_C: track 2.78 -> 184.2 mm, vias 0 -> 4
- net CSense_OUT_LES: track 0.00 -> 139.5 mm, vias 0 -> 1
- net Current Sense_B: track 0.00 -> 132.2 mm, vias 0 -> 4
- net HS_MOS_C: track 9.59 -> 101.7 mm, vias 1 -> 2
- net LS_MOS_C: track 10.9 -> 99.2 mm, vias 1 -> 2
- net Current Sense_A: track 4.68 -> 82.1 mm, vias 0 -> 3
- net BRAKE: track 0.00 -> 75.9 mm, vias 0 -> 1
- net CRUISE: track 0.00 -> 66.7 mm, vias 0 -> 1
- net STATUS_LED: track 0.00 -> 58.5 mm, vias 0 -> 1
- net /FET/LS_MOS_A: track 4.61 -> 60.0 mm, vias 1 -> 2
- net /FET/HS_MOS_A: track 5.82 -> 61.1 mm, vias 1 -> 2
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- added copper zone on B.Cu, net +VDC
- added copper zone on F.Cu, net +VDC
- added copper zone on In1.Cu, net +VDC
- added copper zone on In2.Cu, net +VDC
- added copper zone on In4.Cu, net +VDC
- added copper zone on B.Cu, net -VDC
- added copper zone on F.Cu, net -VDC
- added copper zone on In1.Cu, net -VDC
- added copper zone on In3.Cu, net -VDC
- added copper zone on In4.Cu, net -VDC
- added copper zone on B.Cu, net /FET/Phase_A_FET/PHASE_A
- added copper zone on In1.Cu, net /FET/Phase_A_FET/PHASE_A
- added copper zone on In2.Cu, net /FET/Phase_A_FET/PHASE_A
- added copper zone on In3.Cu, net /FET/Phase_A_FET/PHASE_A
- added copper zone on In4.Cu, net /FET/Phase_A_FET/PHASE_A
- added copper zone on B.Cu, net /FET/Phase_B_FET/PHASE_B
- added copper zone on In1.Cu, net /FET/Phase_B_FET/PHASE_B
- added copper zone on In2.Cu, net /FET/Phase_B_FET/PHASE_B
- added copper zone on In3.Cu, net /FET/Phase_B_FET/PHASE_B
- added copper zone on In4.Cu, net /FET/Phase_B_FET/PHASE_B
- added copper zone on B.Cu, net /FET/Phase_C_FET/PHASE_C
- added copper zone on F.Cu, net /FET/Phase_C_FET/PHASE_C
- added copper zone on In1.Cu, net /FET/Phase_C_FET/PHASE_C
- added copper zone on In2.Cu, net /FET/Phase_C_FET/PHASE_C
- added copper zone on In3.Cu, net /FET/Phase_C_FET/PHASE_C
- added copper zone on In4.Cu, net /FET/Phase_C_FET/PHASE_C
- added copper zone on F.Cu, net Net-(H1-Pad1)
Other:
- board size 207.2 x 164.4 mm -> 119.6 x 167.9 mm
- board text removed: "10R"

Commit message: son update
Parts:
- BZ1: moved to B.Cu
- moved C7 5.53 mm to (99.0, 71.5)
- moved C8 4.03 mm to (93.0, 63.5)
- turned BZ1 to 180 degrees
Routing:
- net CSense_OUT_LES: track 139.5 -> 147.5 mm
Other:
- board text added: "0x616E7368696E7869737468656772656174657374"
- board text added: "0x73766D2E62682E676E636B2E692E6D2E6C0A"
- board text added: "Designed by Anshinx for Pehlivan Team With <3 Yener S. Güneş"
- board text added: "PEHLI SHELL MDU V1"
- board text added: "SEM 2026"

Commit message: bit artık
Parts:
- removed C31, C32: 2.2µF, Capacitor_SMD:C_0603_1608Metric_Pad1.08x0.95mm_HandSolder
- removed C37, C41: 100nF, Capacitor_SMD:C_0603_1608Metric_Pad1.08x0.95mm_HandSolder
- removed C38: 10uF, Capacitor_SMD:C_0603_1608Metric_Pad1.08x0.95mm_HandSolder
- removed J10: Conn_01x02, Connector_PinSocket_2.00mm:PinSocket_1x02_P2.00mm_Horizontal
- added H10: MountingHole, MountingHole:MountingHole_2.2mm_M2, F.Cu at (202.7, 180.3)
- added H3: MountingHole, MountingHole:MountingHole_2.2mm_M2, F.Cu at (146.1, 32.2)
- added H8: MountingHole, MountingHole:MountingHole_2.2mm_M2, F.Cu at (94.6, 87.5)
- added H9: MountingHole, MountingHole:MountingHole_2.2mm_M2, F.Cu at (134.9, 184.0)
- added Q2: BC817, Package_TO_SOT_SMD:SOT-23, F.Cu at (104.2, 137.7)
- added R73: 470, Resistor_SMD:R_0603_1608Metric_Pad0.98x0.95mm_HandSolder, F.Cu at (109.6, 139.6)
- BZ1, J1, NT9: moved to F.Cu
- C33, C34, C35, C51, C52, C53, C54, C55, C56, NT4, NT7, R14, R15, R16, R17, R18, R19, R20, R23, R24, R25, R7, U12: moved to B.Cu
- JP1: footprint Connector_PinHeader_1.27mm:PinHeader_1x03_P1.27mm_Horizontal -> Connector_PinHeader_1.27mm:PinHeader_1x03_P1.27mm_Vertical
- NT6: footprint NetTie:NetTie-2_SMD_Pad0.5mm -> NetTie:NetTie-2_SMD_Pad2.0mm
- R12: footprint Resistor_THT:R_Axial_DIN0207_L6.3mm_D2.5mm_P7.62mm_Horizontal -> Resistor_SMD:R_0603_1608Metric
- U1: value STM32F205VGTx -> STM32G474VETx
- moved NT6 79.9 mm to (136.8, 89.5), turned to -90 degrees
- moved J7 77.1 mm to (103.0, 186.2), turned to 90 degrees
- moved J12 64.7 mm to (97.9, 186.2), turned to 90 degrees
- moved J3 62.1 mm to (91.6, 120.1)
- moved R22 61.9 mm to (94.2, 121.1), turned to -90 degrees
- moved U8 59.8 mm to (107.5, 122.3)
- moved C36 58.8 mm to (105.8, 118.6), turned to 0 degrees
- moved C45 57.7 mm to (114.2, 121.6), turned to 0 degrees
- moved SW1 51.3 mm to (91.7, 163.6), turned to 90 degrees
- moved SW2 50.4 mm to (125.5, 130.6), turned to -90 degrees
- moved C28 47.0 mm to (93.1, 168.0), turned to 0 degrees
- moved R11 45.9 mm to (97.1, 116.6)
- moved D2 42.9 mm to (92.8, 114.2), turned to 0 degrees
- moved J6 42.7 mm to (135.9, 147.3)
- moved J5 42.4 mm to (131.8, 138.1), turned to 0 degrees
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Connections:
- JP1 pad 1: STATUS_LED -> Net-(JP1-A)
- NT6 pad 1: +3V3 -> -VDC
- NT6 pad 2: VDD_6 -> GND
- R22 pad 1: Net-(J3-Pin_2) -> Net-(J3-Pin_1)
- R22 pad 2: Net-(J3-Pin_1) -> Net-(J3-Pin_2)
- U1 pad 10: GND -> unconnected-(U1-PF9-Pad10)
- U1 pad 100: VDD_6 -> VDD_5
- U1 pad 11: VDD_1 -> unconnected-(U1-PF10-Pad11)
- U1 pad 15: unconnected-(U1-PC0-Pad15) -> TMP_SDA
- U1 pad 16: unconnected-(U1-PC1-Pad16) -> TMP_SCL
- U1 pad 17: unconnected-(U1-PC2-Pad17) -> Current Sense_B
- U1 pad 18: unconnected-(U1-PC3-Pad18) -> TMP_ALERT
- U1 pad 19: VDD_2 -> unconnected-(U1-PF2-Pad19)
- U1 pad 2: CRUISE -> unconnected-(U1-PE3-Pad2)
- U1 pad 20: GND -> CSense_OUT_LES
- U1 pad 21: VREF+ -> B_VOL_CHECK
- U1 pad 22: VREF+ -> ACCEL
- U1 pad 23: CSense_OUT_LES -> GND
- U1 pad 24: B_VOL_CHECK -> VDD_1
- U1 pad 25: ACCEL -> TEMP_SENSOR
- U1 pad 26: TEMP_SENSOR -> REGEN
- U1 pad 27: GND -> unconnected-(U1-PA5-Pad27)
- U1 pad 28: VDD_3 -> Current Sense_A
- U1 pad 29: REGEN -> unconnected-(U1-PA7-Pad29)
- U1 pad 31: Current Sense_A -> unconnected-(U1-PC5-Pad31)
- U1 pad 32: Current Sense_B -> Current_Sense_C
- U1 pad 35: Current_Sense_C -> GND
- U1 pad 36: unconnected-(U1-PB1-Pad36) -> VREF+
- U1 pad 37: unconnected-(U1-PB2-Pad37) -> VREF+
- U1 pad 47: CAN_S -> BT_TX
- U1 pad 48: BT_TX -> GND
- U1 pad 49: Net-(U1-VCAP_1) -> VDD_2
- U1 pad 50: VDD_4 -> BT_RX
- U1 pad 51: BT_RX -> BT_KEY
- U1 pad 52: BT_KEY -> unconnected-(U1-PB13-Pad52)
- U1 pad 63: HALL_A -> GND
- U1 pad 64: HALL_B -> VDD_3
- U1 pad 65: HALL_C -> HALL_A
- U1 pad 66: BT_STATE -> HALL_B
- U1 pad 67: Current Sense_C -> HALL_C
- U1 pad 68: unconnected-(U1-PA9-Pad68) -> BT_STATE
- U1 pad 70: D- -> unconnected-(U1-PA9-Pad70)
- U1 pad 71: D+ -> unconnected-(U1-PA10-Pad71)
- U1 pad 72: SWDIO -> D-
- U1 pad 73: Net-(U1-VCAP_2) -> D+
- U1 pad 75: VDD_5 -> VDD_4
- U1 pad 76: SWCLK -> SWDIO
- U1 pad 77: unconnected-(U1-PA15-Pad77) -> SWCLK
- U1 pad 81: TMP_SCL -> unconnected-(U1-PC12-Pad81)
- U1 pad 82: TMP_SDA -> CAN_TX
- U1 pad 83: TMP_ALERT -> CAN_RX
- U1 pad 92: /MCU/I2C_SCL -> unconnected-(U1-PB5-Pad92)
- U1 pad 93: /MCU/I2C_SDA -> /MCU/I2C_SCL
- U1 pad 94: /MCU/BOOT0 -> /MCU/I2C_SDA
- U1 pad 95: CAN_RX -> /MCU/BOOT0
- U1 pad 96: CAN_TX -> unconnected-(U1-PB9-Pad96)
- U1 pad 97: STATUS_LED -> BUZZER
- U1 pad 98: BUZZER -> STATUS_LED
- U1 pad 99: unconnected-(U1-RFU-Pad99) -> GND
- U11 pad 5: Current Sense_C -> Current_Sense_C
- U8 pad 6: Net-(J3-Pin_2) -> Net-(J3-Pin_1)
- U8 pad 7: Net-(J3-Pin_1) -> Net-(J3-Pin_2)
- U8 pad 8: CAN_S -> GND
Routing:
- net Current_Sense_C: track 0.00 -> 200.7 mm, vias 0 -> 4
- net Current Sense_C: track 184.2 -> 0.00 mm, vias 4 -> 0
- net GND: track 465.5 -> 585.4 mm, vias 29 -> 52
- net CRUISE: track 66.7 -> 0.00 mm, vias 1 -> 0
- net STATUS_LED: track 58.5 -> 2.64 mm, vias 1 -> 0
- net +5V: track 211.2 -> 258.3 mm, vias 2 -> 5
- net +12V: track 243.8 -> 197.8 mm, vias 5 -> 7
- net CAN_S: track 39.1 -> 0.00 mm, vias 3 -> 0
- net -VDC: track 115.5 -> 76.8 mm, vias 648 -> 673
- net Net-(J2-Pin_1): track 13.4 -> 44.9 mm
- net D-: track 9.63 -> 41.1 mm, vias 0 -> 2
- net Current Sense_B: track 132.2 -> 163.4 mm
- net LS_MOS_C: track 99.2 -> 130.3 mm
- net +3V3: track 110.9 -> 141.4 mm, vias 6 -> 15
- net D+: track 9.60 -> 39.3 mm, vias 0 -> 2
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- added copper zone on In3.Cu, net +3V3
- added copper zone on In2.Cu, net -VDC
- added copper zone on B.Cu, net GND
- added copper zone on F.Cu, net GND
- added copper zone on In2.Cu, net GND
- added copper zone on In3.Cu, net GND
- added copper zone on In4.Cu, net GND
- removed copper zone on F.Cu, net +3V3
Other:
- board text removed: "Designed by Anshinx for Pehlivan Team With <3 Yener S. Güneş"
- board text removed: "PEHLI SHELL MDU V1"
