File: Motor_Driver_Shell_Eco.kicad_pcb (KiCad board)
At the start: 4 copper layers, 165.9 x 127.7 mm, 210 parts, among them J1 I2C EKRAN, J11 USB_C_Receptacle, J12 Conn_01x02, J13 OUTSIDE LED, J2 HALL INPUT, J3 Conn_01x02, J4 Conn_01x02, J5 Conn_01x04, J7 Conn_01x02, J8 Conn_01x03, J9 Conn_01x03, Q1 BC817, Q14 IAUS300N08S5N0, Q15 IAUS300N08S5N0, Q16 IAUS300N08S5N0, Q17 IAUS300N08S5N0, Q18 IAUS300N08S5N0, Q19 IAUS300N08S5N0, Q2 BC817, Q20 IAUS300N08S5N0, Q21 IAUS300N08S5N0, Q6 IAUS300N08S5N0, Q7 IAUS300N08S5N0, Q8 IAUS300N08S5N0, Q9 IAUS300N08S5N0, SW1 SW_Push, SW2 SW_Push, U1 STM32G474VETx, U10 IRS21867S, U11 INA241A2, U12 XC6206 - 3V3, U13 INA241A2, U14 AP2204K-5.0, U2 LM5017MR, U3 AP2204K-5.0, U4 XC6206 - 3V3, U5 INA241A2, U6 IRS21867S, U8 TJA1051T, U9 IRS21867S, Y1 8MHz

Commit message: MD DONE IHOPE
Connections:
- U9 pad 4: unconnected-(U9-COM-Pad4) -> -VDC
Routing:
- net GND: track 60.9 -> 74.5 mm
- net Net-(U2-SW): track 6.31 -> 14.3 mm, vias 0 -> 2
- net Net-(Q19-Pad2): track 0.00 -> 4.78 mm, vias 14 -> 15
- net Net-(D4-K): track 6.93 -> 9.73 mm
- net -VDC: vias 528 -> 527
Other:
- board text added: "A"
- board text added: "B"
- board text added: "C"
Changed lines of the file:
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@@
 	(net 167 "Net-(Q16-Pad2)")
 	(net 168 "Net-(Q19-Pad2)")
-	(net 169 "unconnected-(U9-COM-Pad4)")
 	(footprint "Resistor_SMD:R_0603_1608Metric"
 		(layer "F.Cu")
@@
 			(layers "B.Cu" "B.Mask" "B.Paste")
 			(roundrect_rratio 0.25)
-			(net 169 "unconnected-(U9-COM-Pad4)")
+			(net 120 "-VDC")
 			(pinfunction "COM")
 			(pintype "power_in")
@@
 		)
 	)
+	(gr_text "C"
+		(at 134.08 152.53 0)
+		(layer "F.SilkS")
+		(effects
+			(font
+				(size 3 3)
+				(thickness 0.75)
+				(bold yes)
+			)
+			(justify left bottom)
+		)
+	)
 	(gr_text "REGENERATIVE\nBRAKE\n"
 		(at 47.5 49 270)
@@
 		)
 	)
+	(gr_text "B"
+		(at 97.88 151.82 0)
+		(layer "F.SilkS")
+		(effects
+			(font
+				(size 3 3)
+				(thickness 0.75)
+				(bold yes)
+			)
+			(justify left bottom)
+		)
+	)
+	(gr_text "A\n"
+		(at 60.63 152.11 0)
+		(layer "F.SilkS")
+		(effects
+			(font
+				(size 3 3)
+				(thickness 0.75)
+				(bold yes)
+			)
+			(justify left bottom)
+		)
+	)
 	(gr_text "BOOT0\n"
 		(at 65.184277 38.12 0)
@@
 	)
 	(segment
+		(start 163.025 73.25)
+		(end 163.275 73.5)
+		(width 0.8)
+		(layer "F.Cu")
+		(net 4)
+	)
+	(segment
+		(start 163.275 73.5)
+		(end 163.275 75.335)
+		(width 0.8)
+		(layer "F.Cu")
+		(net 4)
+	)
+	(segment
 		(start 169.8 70.175)
 		(end 169.725 70.1)
@@
 	)
 	(segment
-		(start 163.275 75.335)
-		(end 163.275 73.5)
+		(start 169.725 70.1)
+		(end 169.725 67.825)
 		(width 0.8)
 		(layer "F.Cu")
@@
 	)
 	(segment
-		(start 169.725 70.1)
-		(end 169.725 67.825)
+		(start 169.8 71.6)
+		(end 169.8 70.175)
 		(width 0.8)
 		(layer "F.Cu")
@@
 	)
 	(segment
-		(start 163.275 73.5)
+		(start 162.775 73.25)
 		(end 163.025 73.25)
 		(width 0.8)
@@
 		(net 4)
 	)
+	(via
+		(at 169.8 71.6)
+		(size 0.6)
+		(drill 0.3)
+		(layers "F.Cu" "B.Cu")
+		(net 4)
+	)
+	(via
+		(at 162.775 73.25)
+		(size 0.6)
+		(drill 0.3)
+		(layers "F.Cu" "B.Cu")
+		(net 4)
+	)
 	(segment
-		(start 169.8 71.6)
-		(end 169.8 70.175)
+		(start 162.775 73.25)
+		(end 164.425 71.6)
 		(width 0.8)
-		(layer "F.Cu")
+		(layer "B.Cu")
+		(net 4)
+	)
+	(segment
+		(start 164.425 71.6)
+		(end 169.8 71.6)
+		(width 0.8)
+		(layer "B.Cu")
 		(net 4)
 	)
@@
 	)
 	(segment
+		(start 75.66 39.975)
+		(end 75.085 39.4)
+		(width 0.5)
+		(layer "F.Cu")
+		(net 111)
+	)
+	(segment
+		(start 83.725 39.4)
+		(end 83.725 35.22)
+		(width 0.5)
+		(layer "F.Cu")
+		(net 111)
+	)
+	(segment
 		(start 63.434277 69.645)
 		(end 63.434277 66.634277)
@@
 	)
 	(segment
+		(start 74.88 41.87)
+		(end 74.88 39.605)
+		(width 1)
+		(layer "F.Cu")
+		(net 111)
+	)
+	(segment
 		(start 84.834277 51.11)
 		(end 84.834277 50.670723)
@@
 	)
 	(segment
+		(start 83.18 39.4)
+		(end 82.605 39.975)
+		(width 0.5)
+		(layer "F.Cu")
+		(net 111)
+	)
+	(segment
 		(start 71.064277 57.1)
 		(end 71.694277 56.47)
@@
 	)
 	(segment
+		(start 76.205 39.975)
+		(end 75.66 39.975)
+		(width 0.5)
+		(layer "F.Cu")
+		(net 111)
+	)
+	(segment
 		(start 58.065777 52.489)
 		(end 57.459277 51.8825)
@@
 	)
 	(segment
+		(start 83.725 39.4)
+		(end 83.18 39.4)
+		(width 0.5)
+		(layer "F.Cu")
+		(net 111)
+	)
+	(segment
 		(start 59.434277 53.17219)
 		(end 58.751087 52.489)
@@
 	)
 	(segment
+		(start 74.88 39.605)
+		(end 75.085 39.4)
+		(width 1)
+		(layer "F.Cu")
+		(net 111)
+	)
+	(segment
 		(start 85.645 40.89)
 		(end 84.625 41.91)
@@
 		(net 111)
 	)
+	(segment
+		(start 75.085 39.4)
+		(end 75.085 35.22)
+		(width 0.5)
+		(layer "F.Cu")
+		(net 111)
+	)
 	(via
 		(at 57.584277 46.87)
@@
 	)
 	(via
-		(at 84.065 130.65)
-		(size 0.6)
-		(drill 0.3)
-		(layers "F.Cu" "B.Cu")
-		(net 120)
-	)
-	(via
 		(at 137.615 87.9)
 		(size 0.6)
@@
 	)
 	(segment
+		(start 84.435908 120.864235)
+		(end 84.935908 121.364235)
+		(width 0.5)
+		(layer "B.Cu")
+		(net 124)
+	)
+	(segment
 		(start 84.935908 126.674235)
 		(end 84.935908 121.364235)
@@
 	)
 	(segment
+		(start 82.345908 120.864235)
+		(end 84.435908 120.864235)
+		(width 0.5)
+		(layer "B.Cu")
+		(net 124)
+	)
+	(segment
 		(start 121.458929 126.066832)
 		(end 121.488929 126.036832)
@@
 		(net 167)
 	)
+	(segment
+		(start 157.165 135.295)
+		(end 157.165 135.965)
+		(width 0.5)
+		(layer "F.Cu")
+		(net 168)
+	)
+	(segment
+		(start 157.2 136)
+		(end 157.165 135.965)
+		(width 0.5)
+		(layer "F.Cu")
+		(net 168)
+	)
 	(via
 		(at 135.178929 135.786832)
@@
 	)
 	(via
+		(at 157.2 136)
+		(size 0.6)
+		(drill 0.3)
+		(layers "F.Cu" "B.Cu")
+		(net 168)
+	)
+	(via
 		(at 148.478929 135.836832)
 		(size 0.6)
@@
 		(net 168)
 	)
+	(segment
+		(start 155.155 135.95)
+		(end 159.215 135.95)
+		(width 0.5)
+		(layer "B.Cu")
+		(net 168)
+	)
