File: mosfets.kicad_sch (KiCad schematic)
At the start: 38 parts, among them Q10 IXTP90N15T, Q11 IXTP90N15T, Q12 IXTP90N15T, Q13 IXTP90N15T, U10 IRS21867S, U6 IRS21867S, U7 IR2110, U9 IRS21867S

Commit message: rev3
Parts:
- removed C58, C59, C60: 100uf, Capacitor_SMD:C_0805_2012Metric_Pad1.18x1.45mm_HandSolder, symbol Device:C
- C39, C40, C57: footprint Capacitor_THT:C_Rect_L7.2mm_W3.5mm_P5.00mm_FKS2_FKP2_MKS2_MKP2 -> Capacitor_SMD:C_1210_3225Metric_Pad1.33x2.70mm_HandSolder
Connections:
- net -VDC: now also C88.2, C89.2, C90.2, U10.4 (COM), U6.4 (COM)
- net GND: no longer C88.2, C89.2, C90.2, U10.4 (COM), U6.4 (COM), U9.4 (COM)
Other:
- moved on the sheet: C57

Commit message: MD DONE IHOPE
Connections:
- net -VDC: now also U9.4 (COM)
Changed lines of the file:
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@@
 	(symbol
 		(lib_id "power:-VDC")
-		(at 53.34 52.2329 180)
+		(at 53.34 52.07 180)
 		(unit 1)
 		(exclude_from_sim no)
@@
 		(fields_autoplaced yes)
 		(property "Reference" "#PWR0101"
-			(at 53.34 49.6929 0)
+			(at 53.34 49.53 0)
 			(effects
 				(font
@@
 		)
 		(property "Value" "-VDC"
-			(at 53.34 59.8529 0)
+			(at 53.34 59.69 0)
 			(effects
 				(font
@@
 		)
 		(property "Footprint" ""
-			(at 53.34 52.2329 0)
+			(at 53.34 52.07 0)
 			(effects
 				(font
@@
 		)
 		(property "Datasheet" ""
-			(at 53.34 52.2329 0)
+			(at 53.34 52.07 0)
 			(effects
 				(font
@@
 		)
 		(property "Description" "Power symbol creates a global label with name \"-VDC\""
-			(at 53.34 52.2329 0)
+			(at 53.34 52.07 0)
 			(effects
 				(font
